Commit message: added imu rpy configuration in urdf description

File: amiga_ros2_description/urdf/amiga_descr.urdf.xacro (robot description, xacro)
@@ -41,14 +41,17 @@
   <xacro:gps
     parent_link="base_link"
-    gps_link_name="GPS_link"
+    gps_link_name="gps_link"
     joint_origin_xyz="-0.343 0.27301 1.0163"
     joint_origin_rpy="0 0 0"/>
   <!-- Cameras -->
   <!-- Front -->
+  <!-- imu_rpy="3.14159265359 1.5708 0" -->
+  <xacro:property name="oak0_offset" value="${62.2 * pi / 180}"/>
   <xacro:oak_d_w_poe
     camera_name="oak0"
     parent_link="base_link"
     mount_origin_xyz="-0.24835 0.27301 0.95145"
-    mount_origin_rpy="3.1416 0.2618 0"/>
+    mount_origin_rpy="${pi} 0.2618 0"
+    imu_rpy="${pi} ${pi/2} 0"/>
   <!-- Back -->
   <xacro:oak_d_w_poe
@@ -56,4 +59,5 @@
     parent_link="base_link"
     mount_origin_xyz="-0.43765 0.27301 0.95145"
-    mount_origin_rpy="-3.1416 0.2618 -3.1416"/>
+    mount_origin_rpy="-${pi} 0.2618 -${pi}"
+    imu_rpy="${pi} ${pi/2} 0"/>
 </robot>

File: amiga_ros2_description/urdf/oak_d_w_poe.urdf.xacro (robot description, xacro)
@@ -2,5 +2,5 @@
 <robot xmlns:xacro="http://ros.org/wiki/xacro">
   <!-- Based on: https://github.com/luxonis/depthai-ros/tree/humble/depthai_descriptions -->
-  <xacro:macro name="oak_d_w_poe" params="camera_name parent_link mount_origin_xyz mount_origin_rpy">
+  <xacro:macro name="oak_d_w_poe" params="camera_name parent_link mount_origin_xyz mount_origin_rpy imu_rpy">
     <!-- Mount link -->
     <link name="${camera_name}_mount_link"/>
@@ -61,5 +61,6 @@
       <parent link="${camera_name}_base_link"/>
       <child link="${camera_name}_imu_frame"/>
-      <origin xyz="-0.008 0.04 0.020265" rpy="3.14159265359 1.5708 0"/>
+      <!-- <origin xyz="-0.008 0.04 0.020265" rpy="3.14159265359 1.5708 0"/> -->
+      <origin xyz="-0.008 0.04 0.020265" rpy="${imu_rpy}"/>
     </joint>
   </xacro:macro>
