Commit message: fixed issues with urdf

File: amiga_ros2_description/urdf/base.urdf.xacro (robot description, xacro)
@@ -9,8 +9,8 @@
     <link name="base_link"/>
     <!-- Fixed joint from footprint to base_link -->
-    <joint name="base_to_footprint" type="fixed">
-      <parent link="base_footprint"/>
-      <child link="base_link"/>
-      <origin xyz="0 0 ${vertical_offset}" rpy="0 0 0"/>
+    <joint name="base_footprint_joint" type="fixed">
+      <parent link="base_link"/>
+      <child link="base_footprint"/>
+      <origin xyz="0 0 -${vertical_offset}" rpy="0 0 0"/>
     </joint>
   </xacro:macro>

File: amiga_ros2_description/urdf/oak_d_w_poe.urdf.xacro (robot description, xacro)
@@ -22,5 +22,6 @@
       <parent link="${camera_name}_base_link"/>
       <child link="${camera_name}_rgb_camera_frame"/>
-      <origin xyz="0 0 0" rpy="0 0 0"/>
+      <!-- <origin xyz="0 0 0" rpy="0 0 0"/> -->
+      <origin xyz="0 0 0" rpy="3.14159 0 0"/>
     </joint>
     <link name="${camera_name}_rgb_camera_optical_frame"/>
@@ -35,5 +36,6 @@
       <parent link="${camera_name}_base_link"/>
       <child link="${camera_name}_left_camera_frame"/>
-      <origin xyz="0 -0.0375 0" rpy="0 0 0"/>
+      <!-- <origin xyz="0 -0.0375 0" rpy="0 0 0"/> -->
+      <origin xyz="0 -0.0375 0" rpy="3.14159 0 0"/>
     </joint>
     <link name="${camera_name}_left_camera_optical_frame"/>
@@ -48,5 +50,6 @@
       <parent link="${camera_name}_base_link"/>
       <child link="${camera_name}_right_camera_frame"/>
-      <origin xyz="0 0.0375 0" rpy="0 0 0"/>
+      <!-- <origin xyz="0 0.0375 0" rpy="0 0 0"/> -->
+      <origin xyz="0 0.0375 0" rpy="3.14159 0 0"/>
     </joint>
     <link name="${camera_name}_right_camera_optical_frame"/>
